File: MotorSpeedController/Hardware/MotorSpeedController.brd (EAGLE design)
At the start: 51.2 x 29.2 mm, 49 parts, among them IC1 MIC5219 5V, IC2 ATMEGA32U4-AU, J1 POWER, J2 MOTOR, J3 USB MICRO, J4 I2C, J5 PROG, Q1 16MHz

Commit message: Add custom library.
Parts:
- J3: device NidecController:MICROBUILDER_4UCONN_20329_V2 -> CrazyGiraffe-MotorSpeedController:MICROBUILDER_4UCONN_20329_V2
Changed lines of the file:
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@@
 <attribute name="VALUE" x="21.463" y="5.334" size="1.27" layer="27" ratio="10" rot="R270"/>
 </element>
-<element name="J3" library="NidecController" package="MICROBUILDER_4UCONN_20329_V2" value="USB MICRO" x="5.588" y="23.749" smashed="yes" rot="R180">
+<element name="J3" library="CrazyGiraffe-MotorSpeedController" package="MICROBUILDER_4UCONN_20329_V2" value="USB MICRO" x="5.588" y="23.749" smashed="yes" rot="R180">
 <attribute name="NAME" x="10.906" y="28.204" size="0.6096" layer="25" ratio="18" rot="R180"/>
 <attribute name="VALUE" x="8.366" y="30.159" size="0.4064" layer="27" ratio="10" rot="R180"/>
