File: MotorSpeedController/Hardware/MotorSpeedController.sch (EAGLE design)
At the start: 47 parts, among them IC1 MIC5219 5V, IC2 ATMEGA32U4-AU, J1 POWER, J2 MOTOR, J3 USB MICRO, J4 I2C, J5 PROG, Q1 16MHz

Commit message: Add custom library.
Parts:
- J3: device NidecController:MICROBUILDER_USB_MICRO_20329_V2 -> CrazyGiraffe-MotorSpeedController:MICROBUILDER_USB_MICRO_20329_V2
Changed lines of the file:
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@@
 <part name="C11" library="adafruit" library_urn="urn:adsk.eagle:library:420" deviceset="C-US" device="025-030X050" package3d_urn="urn:adsk.eagle:package:6240322/1" value="20pF"/>
 <part name="C12" library="adafruit" library_urn="urn:adsk.eagle:library:420" deviceset="C-US" device="025-030X050" package3d_urn="urn:adsk.eagle:package:6240322/1" value="20pF"/>
-<part name="J3" library="NidecController" deviceset="MICROBUILDER_USB" device="_MICRO_20329_V2" value="USB MICRO"/>
+<part name="J3" library="CrazyGiraffe-MotorSpeedController" deviceset="MICROBUILDER_USB" device="_MICRO_20329_V2" value="USB MICRO"/>
 <part name="R15" library="rcl" library_urn="urn:adsk.eagle:library:334" deviceset="R-TRIMM" device="3296Y" package3d_urn="urn:adsk.eagle:package:26036/1" value="10k"/>
 </parts>
