File: hardware/MotorSpeedController/MotorSpeedController.sch (EAGLE design)
At the start: 47 parts, among them IC1 MIC5219 5V, IC2 ATMEGA32U4-AU, J1 POWER, J2 MOTOR, J3 USB MICRO, J4 I2C, J5 PROG, Q1 16MHz

Commit message: Add I2C interrupt/IO.
Parts:
- added R7: 4.7k, rcl:R-US_R0603
- J4: device pinhead:PINHD-1X4 -> pinhead:PINHD-1X5
Connections:
- new net INT: IC2.PD4(ICP1/ADC8), R7.1
- new net N$8: J4.5, R7.2
Changed lines of the file:
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@@
 <attribute name="SPICEPREFIX" value="E"/>
 </part>
-<part name="J4" library="pinhead" library_urn="urn:adsk.eagle:library:325" deviceset="PINHD-1X4" device="" package3d_urn="urn:adsk.eagle:package:22407/2" value="I2C"/>
+<part name="J4" library="pinhead" library_urn="urn:adsk.eagle:library:325" deviceset="PINHD-1X5" device="" package3d_urn="urn:adsk.eagle:package:22469/2" value="I2C"/>
 <part name="IC2" library="adafruit" library_urn="urn:adsk.eagle:library:420" deviceset="ATMEGA32U4" device="-AU" package3d_urn="urn:adsk.eagle:package:6240644/1"/>
 <part name="C8" library="SparkFun-Passives" deviceset="CAP" device="0603-CAP" value=".1uF"/>
@@
 <part name="J3" library="CrazyGiraffe-MotorSpeedController" deviceset="MICROBUILDER_USB" device="_MICRO_20329_V2" value="USB MICRO"/>
 <part name="R15" library="rcl" library_urn="urn:adsk.eagle:library:334" deviceset="R-TRIMM" device="3296Y" package3d_urn="urn:adsk.eagle:package:26036/1" value="10k"/>
+<part name="R7" library="rcl" library_urn="urn:adsk.eagle:library:334" deviceset="R-US_" device="R0603" package3d_urn="urn:adsk.eagle:package:23555/3" value="4.7k"/>
 </parts>
 <sheets>
@@
 <attribute name="VALUE" x="175.26" y="154.94" size="1.778" layer="96" rot="MR90"/>
 </instance>
-<instance part="GND9" gate="1" x="200.66" y="137.16" smashed="yes" rot="MR0">
-<attribute name="VALUE" x="203.2" y="134.62" size="1.778" layer="96" rot="MR0"/>
+<instance part="GND9" gate="1" x="200.66" y="132.08" smashed="yes" rot="MR0">
+<attribute name="VALUE" x="203.2" y="129.54" size="1.778" layer="96" rot="MR0"/>
 </instance>
 <instance part="R5" gate="G$1" x="190.5" y="157.48" smashed="yes" rot="MR270">
@@
 <attribute name="NAME" x="42.291" y="62.23" size="1.778" layer="95" rot="MR270"/>
 <attribute name="VALUE" x="44.45" y="62.23" size="1.778" layer="96" rot="MR270"/>
+</instance>
+<instance part="R7" gate="G$1" x="190.5" y="139.7" smashed="yes" rot="MR180">
+<attribute name="NAME" x="186.69" y="138.2014" size="1.778" layer="95" rot="MR180"/>
+<attribute name="VALUE" x="191.77" y="143.002" size="1.778" layer="96" rot="MR180"/>
 </instance>
 </instances>
@@
 </segment>
 </bus>
-<bus name="I2C:SCL,SDA">
+<bus name="I2C:INT,SCL,SDA">
 <segment>
 <wire x1="180.34" y1="149.86" x2="180.34" y2="142.24" width="0.762" layer="92"/>
@@
 <segment>
 <pinref part="GND9" gate="1" pin="GND"/>
+<wire x1="200.66" y1="142.24" x2="200.66" y2="134.62" width="0.1524" layer="91"/>
+<pinref part="J4" gate="A" pin="4"/>
 <wire x1="208.28" y1="142.24" x2="200.66" y2="142.24" width="0.1524" layer="91"/>
-<wire x1="200.66" y1="142.24" x2="200.66" y2="139.7" width="0.1524" layer="91"/>
-<pinref part="J4" gate="A" pin="4"/>
 </segment>
 <segment>
@@
 <segment>
 <pinref part="P+4" gate="1" pin="+5V"/>
-<pinref part="J4" gate="A" pin="3"/>
-<wire x1="208.28" y1="144.78" x2="200.66" y2="144.78" width="0.1524" layer="91"/>
 <wire x1="200.66" y1="144.78" x2="200.66" y2="165.1" width="0.1524" layer="91"/>
 <pinref part="R5" gate="G$1" pin="1"/>
@@
 <wire x1="195.58" y1="162.56" x2="195.58" y2="165.1" width="0.1524" layer="91"/>
 <junction x="195.58" y="165.1"/>
+<pinref part="J4" gate="A" pin="3"/>
+<wire x1="208.28" y1="144.78" x2="200.66" y2="144.78" width="0.1524" layer="91"/>
 </segment>
 <segment>
@@
 </segment>
 </net>
+<net name="INT" class="0">
+<segment>
+<pinref part="IC2" gate="G$1" pin="PD4(ICP1/ADC8)"/>
+<wire x1="180.34" y1="53.34" x2="165.1" y2="53.34" width="0.1524" layer="91"/>
+<label x="165.862" y="53.594" size="1.778" layer="95"/>
+</segment>
+<segment>
+<pinref part="R7" gate="G$1" pin="1"/>
+<wire x1="180.34" y1="139.7" x2="185.42" y2="139.7" width="0.1524" layer="91"/>
+<label x="181.864" y="139.954" size="1.778" layer="95"/>
+</segment>
+</net>
+<net name="N$8" class="0">
+<segment>
+<pinref part="R7" gate="G$1" pin="2"/>
+<pinref part="J4" gate="A" pin="5"/>
+<wire x1="195.58" y1="139.7" x2="208.28" y2="139.7" width="0.1524" layer="91"/>
+</segment>
+</net>

Commit message: Change footprints to match ordered parts. Put some space between crystal and ICSP. Increase clearance on PWR trace.
Parts:
- C11, C12: value 20pF -> 22pF; device adafruit:C-US025-030X050 -> SparkFun-Capacitors:22PF-0603-50V-5%
- R15: device rcl:R-TRIMM3296Y -> rcl:R-TRIMM3296W
Changed lines of the file:
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@@
 <class number="3" name="diff pairs" width="0.1524" drill="0">
+</class>
+<class number="4" name="vcc_wide" width="0.508" drill="0">
+<clearance class="4" value="0.254"/>
 </class>
 </classes>
@@
 <part name="H2" library="holes" library_urn="urn:adsk.eagle:library:237" deviceset="MOUNT-PAD-ROUND" device="2.8" package3d_urn="urn:adsk.eagle:package:14281/1"/>
 <part name="Q1" library="adafruit" library_urn="urn:adsk.eagle:library:420" deviceset="CRYSTAL" device="HC49S" package3d_urn="urn:adsk.eagle:package:6240901/1" value="16MHz"/>
-<part name="C11" library="adafruit" library_urn="urn:adsk.eagle:library:420" deviceset="C-US" device="025-030X050" package3d_urn="urn:adsk.eagle:package:6240322/1" value="20pF"/>
-<part name="C12" library="adafruit" library_urn="urn:adsk.eagle:library:420" deviceset="C-US" device="025-030X050" package3d_urn="urn:adsk.eagle:package:6240322/1" value="20pF"/>
+<part name="C11" library="SparkFun-Capacitors" library_urn="urn:adsk.eagle:library:510" deviceset="22PF" device="-0603-50V-5%" package3d_urn="urn:adsk.eagle:package:37414/1" value="22pF"/>
+<part name="C12" library="SparkFun-Capacitors" library_urn="urn:adsk.eagle:library:510" deviceset="22PF" device="-0603-50V-5%" package3d_urn="urn:adsk.eagle:package:37414/1" value="22pF"/>
 <part name="J3" library="CrazyGiraffe-MotorSpeedController" deviceset="MICROBUILDER_USB" device="_MICRO_20329_V2" value="USB MICRO"/>
-<part name="R15" library="rcl" library_urn="urn:adsk.eagle:library:334" deviceset="R-TRIMM" device="3296Y" package3d_urn="urn:adsk.eagle:package:26036/1" value="10k"/>
+<part name="R15" library="rcl" library_urn="urn:adsk.eagle:library:334" deviceset="R-TRIMM" device="3296W" package3d_urn="urn:adsk.eagle:package:26033/1" value="10k"/>
 <part name="R7" library="rcl" library_urn="urn:adsk.eagle:library:334" deviceset="R-US_" device="R0603" package3d_urn="urn:adsk.eagle:package:23555/3" value="4.7k"/>
 </parts>
@@
 <attribute name="VALUE" x="109.22" y="67.818" size="1.778" layer="96" rot="R180"/>
 </instance>
-<instance part="C11" gate="G$1" x="99.06" y="63.5" smashed="yes" rot="MR0">
-<attribute name="NAME" x="98.044" y="64.135" size="1.778" layer="95" rot="MR0"/>
-<attribute name="VALUE" x="98.044" y="59.309" size="1.778" layer="96" rot="MR0"/>
-</instance>
-<instance part="C12" gate="G$1" x="106.68" y="58.42" smashed="yes" rot="MR0">
-<attribute name="NAME" x="105.664" y="59.055" size="1.778" layer="95" rot="MR0"/>
-<attribute name="VALUE" x="105.664" y="54.229" size="1.778" layer="96" rot="MR0"/>
+<instance part="C11" gate="G$1" x="99.06" y="60.96" smashed="yes" rot="MR0">
+<attribute name="NAME" x="98.044" y="63.881" size="1.778" layer="95" rot="MR0"/>
+<attribute name="VALUE" x="98.044" y="56.769" size="1.778" layer="96" rot="MR0"/>
+</instance>
+<instance part="C12" gate="G$1" x="106.68" y="55.88" smashed="yes" rot="MR0">
+<attribute name="NAME" x="105.918" y="58.547" size="1.778" layer="95" rot="MR0"/>
+<attribute name="VALUE" x="106.172" y="53.721" size="1.778" layer="96" rot="MR0"/>
 </instance>
 <instance part="J3" gate="G$1" x="40.64" y="25.4" smashed="yes">
@@
 </segment>
 </net>
-<net name="+PWR" class="0">
+<net name="+PWR" class="4">
 <segment>
 <pinref part="J2" gate="A" pin="1"/>
@@
 <net name="N$7" class="0">
 <segment>
-<wire x1="106.68" y1="63.5" x2="106.68" y2="60.96" width="0.1524" layer="91"/>
 <pinref part="IC2" gate="G$1" pin="XTAL2"/>
 <wire x1="116.84" y1="63.5" x2="111.76" y2="63.5" width="0.1524" layer="91"/>
+<wire x1="111.76" y1="64.77" x2="111.76" y2="63.5" width="0.1524" layer="91"/>
+<pinref part="Q1" gate="G$1" pin="1"/>
 <wire x1="111.76" y1="63.5" x2="106.68" y2="63.5" width="0.1524" layer="91"/>
-<wire x1="111.76" y1="64.77" x2="111.76" y2="63.5" width="0.1524" layer="91"/>
 <junction x="111.76" y="63.5"/>
 <pinref part="C12" gate="G$1" pin="1"/>
-<pinref part="Q1" gate="G$1" pin="1"/>
-</segment>
-</net>
+<wire x1="106.68" y1="63.5" x2="106.68" y2="60.96" width="0.1524" layer="91"/>
+</segment>
+</net>
